File: hardware/kicad8.0/NONIK0.kicad_pcb (KiCad board)
At the start: 2 copper layers, 55 x 22 mm, 24 parts, among them J1 AVR-UPDI-3, J2 Qwiic/Stemma QT, J3 Test Pads, J4 Test Pads, SW1 SW_SPST, SW2 SW_Push, SW3 SW_Push, U1 LED_HCMS-2915, U2 ATtiny1604-SS, U3 AP3602A

Commit message: pcb fit and finish
Routing:
- net Vled: track 55.4 -> 64.1 mm
- net DOUT: track 81.8 -> 86.1 mm
- net CE: track 28.1 -> 28.7 mm
Changed lines of the file:
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@@
 		(tags "Jumper 2.54mm")
 		(property "Reference" "J4"
-			(at 1.269999 1.920002 360)
+			(at 1.269999 1.920002 0)
 			(layer "B.SilkS")
 			(hide yes)
@@
 		)
 		(property "Value" "Test Pads"
-			(at 2.349999 -2.000001 360)
+			(at 2.349999 -2.000001 0)
 			(layer "B.Fab")
 			(hide yes)
@@
 		)
 		(property "Footprint" "NONIK0:Pads_1x3_2.54mm"
-			(at 0 0 360)
+			(at 0 0 0)
 			(layer "B.Fab")
 			(hide yes)
@@
 		)
 		(property "Datasheet" ""
-			(at 0 0 360)
+			(at 0 0 0)
 			(layer "B.Fab")
 			(hide yes)
@@
 		)
 		(property "Description" "Generic connector, single row, 01x03, script generated"
-			(at 0 0 360)
+			(at 0 0 0)
 			(layer "B.Fab")
 			(hide yes)
@@
 		)
 		(fp_text user "${REFERENCE}"
-			(at 1.269999 1.920002 360)
+			(at 1.269999 1.920002 0)
 			(layer "B.Fab")
 			(effects
@@
 	(footprint "NONIK0:C_0603_1608Metric"
 		(layer "B.Cu")
-		(at 67.6402 29.2989 -90)
+		(at 67.6402 29.2608 -90)
 		(descr "Capacitor SMD 0603 (1608 Metric), square (rectangular) end terminal, IPC_7351 nominal, (Body size source: IPC-SM-782 page 76, https://www.pcb-3d.com/wordpress/wp-content/uploads/ipc-sm-782a_amendment_1_and_2.pdf), generated with kicad-footprint-generator")
 		(tags "capacitor")
@@
 	(footprint "NONIK0:C_0603_1608Metric"
 		(layer "B.Cu")
-		(at 73.1266 29.2989 90)
+		(at 73.1266 29.2608 90)
 		(descr "Capacitor SMD 0603 (1608 Metric), square (rectangular) end terminal, IPC_7351 nominal, (Body size source: IPC-SM-782 page 76, https://www.pcb-3d.com/wordpress/wp-content/uploads/ipc-sm-782a_amendment_1_and_2.pdf), generated with kicad-footprint-generator")
 		(tags "capacitor")
@@
 		(sheetfile "NONIK0.kicad_sch")
 		(attr smd)
-		(fp_circle
-			(center -1.8 1.7)
-			(end -1.7365 1.7)
-			(stroke
-				(width 0.2)
-				(type solid)
-			)
-			(fill none)
-			(layer "B.SilkS")
-		)
 		(fp_line
 			(start -1.9 -1.8)
@@
 	(segment
 		(start 66.4972 25.8953)
-		(end 71.7296 25.8953)
-		(width 0.381)
-		(layer "F.Cu")
-		(net 1)
-	)
-	(segment
-		(start 66.4972 24.8016)
-		(end 66.4972 25.8953)
+		(end 66.4972 24.8016)
 		(width 0.381)
 		(layer "F.Cu")
@@
 	)
 	(segment
-		(start 72.762142 22.9108)
-		(end 71.7296 23.943342)
+		(start 80.2894 25.6032)
+		(end 80.2894 23.749)
 		(width 0.381)
 		(layer "F.Cu")
@@
 	)
 	(segment
-		(start 80.2894 25.6032)
-		(end 80.2894 23.749)
+		(start 76.708 23.749)
+		(end 76.708 22.9362)
 		(width 0.381)
 		(layer "F.Cu")
@@
 	)
 	(segment
-		(start 76.708 22.9108)
-		(end 72.762142 22.9108)
+		(start 71.7296 22.9108)
+		(end 71.7296 25.8953)
 		(width 0.381)
 		(layer "F.Cu")
@@
 	)
 	(segment
-		(start 76.708 23.749)
-		(end 76.708 22.9362)
+		(start 76.708 22.9108)
+		(end 71.7296 22.9108)
 		(width 0.381)
 		(layer "F.Cu")
@@
 	)
 	(segment
-		(start 71.7296 23.943342)
-		(end 71.7296 25.8953)
+		(start 71.7296 25.8953)
+		(end 66.4972 25.8953)
 		(width 0.381)
 		(layer "F.Cu")
@@
 	)
 	(segment
-		(start 67.6402 28.5239)
-		(end 67.6402 29.1592)
-		(width 0.381)
-		(layer "B.Cu")
-		(net 2)
-	)
-	(segment
-		(start 52.7558 32.4216)
-		(end 52.7558 30.607)
+		(start 53.7972 32.4216)
+		(end 53.7972 30.607)
 		(width 0.381)
 		(layer "B.Cu")
@@
 	)
 	(segment
-		(start 52.7558 30.607)
+		(start 53.7972 30.607)
 		(end 49.9872 30.607)
 		(width 0.381)
@@
 	(segment
 		(start 61.4172 32.4216)
-		(end 52.7558 32.4216)
+		(end 53.7972 32.4216)
 		(width 0.381)
 		(layer "B.Cu")
@@
 	)
 	(segment
+		(start 67.6402 28.5239)
+		(end 67.6402 29.1592)
+		(width 0.381)
+		(layer "B.Cu")
+		(net 2)
+	)
+	(segment
 		(start 76.0476 33.3756)
 		(end 85.883242 33.3756)
@@
 	)
 	(segment
-		(start 67.6402 29.1592)
-		(end 68.9102 29.1592)
+		(start 56.2864 19.304)
+		(end 58.8772 19.304)
 		(width 0.381)
 		(layer "B.Cu")
@@
 	)
 	(segment
-		(start 56.2864 19.304)
-		(end 58.8772 19.304)
+		(start 67.6402 29.1592)
+		(end 68.9102 29.1592)
 		(width 0.381)
 		(layer "B.Cu")
@@
 	)
 	(segment
-		(start 96.9772 28.6878)
-		(end 96.9772 35.2806)
+		(start 97.155 28.6878)
+		(end 97.155 35.1536)
+		(width 0.381)
+		(layer "B.Cu")
+		(net 4)
+	)
+	(segment
+		(start 97.155 35.1536)
+		(end 93.3704 35.1536)
 		(width 0.381)
 		(layer "B.Cu")
@@
 	)
 	(segment
-		(start 93.4466 35.2806)
-		(end 93.4466 38.8874)
+		(start 93.3704 35.1536)
+		(end 93.3704 38.9128)
 		(width 0.381)
 		(layer "B.Cu")
@@
 	)
 	(segment
-		(start 93.4466 38.8874)
-		(end 75.3364 38.8874)
-		(width 0.381)
-		(layer "B.Cu")
-		(net 4)
-	)
-	(segment
-		(start 96.9772 35.2806)
-		(end 93.4466 35.2806)
+		(start 93.3704 38.9128)
+		(end 75.3364 38.9128)
 		(width 0.381)
 		(layer "B.Cu")
@@
 	)
 	(segment
-		(start 75.3364 38.8874)
+		(start 75.3364 38.9128)
 		(end 75.3364 29.0556)
 		(width 0.381)
@@
 	)
 	(segment
-		(start 65.278 28.067)
-		(end 65.278 29.591)
+		(start 65.2272 28.067)
+		(end 65.2272 29.591)
 		(width 0.381)
 		(layer "F.Cu")
@@
 	(segment
 		(start 70.358 28.067)
-		(end 65.278 28.067)
+		(end 65.2272 28.067)
 		(width 0.381)
 		(layer "F.Cu")
@@
 	)
 	(segment
-		(start 65.278 29.591)
+		(start 65.2272 29.591)
 		(end 58.8772 29.591)
 		(width 0.381)
@@
 	(segment
 		(start 58.4962 38.9128)
-		(end 59.3344 38.9128)
+		(end 60.4266 38.9128)
 		(width 0.381)
 		(layer "F.Cu")
@@
 	(segment
 		(start 52.5018 38.9128)
-		(end 53.34 38.9128)
+		(end 56.4642 38.9128)
 		(width 0.381)
 		(layer "F.Cu")
@@
 	(segment
 		(start 53.848 34.544)
-		(end 53.848 32.512)
+		(end 58.8772 34.544)
 		(width 0.381)
 		(layer "F.Cu")
@@
 	)
 	(segment
-		(start 58.9788 34.544)
-		(end 58.9788 32.512)
+		(start 53.848 32.4216)
+		(end 53.848 34.544)
 		(width 0.381)
 		(layer "F.Cu")
@@
 	)
 	(segment
-		(start 58.9788 34.544)
-		(end 53.848 34.544)
+		(start 47.4472 31.115)
+		(end 47.4472 32.4216)
 		(width 0.381)
 		(layer "F.Cu")
@@
 	)
 	(segment
-		(start 58.9788 32.512)
-		(end 53.34 32.512)
+		(start 47.4472 32.4216)
+		(end 49.9872 32.4216)
+		(width 0.381)
+		(layer "F.Cu")
+		(net 23)
+	)
+	(segment
+		(start 58.8772 31.115)
+		(end 47.4472 31.115)
 		(width 0.381)
 		(layer "F.Cu")
@@
 	(segment
 		(start 51.2572 32.4216)
-		(end 51.2572 34.5948)
+		(end 53.848 32.4216)
 		(width 0.381)
 		(layer "F.Cu")
@@
 	)
 	(segment
-		(start 49.9364 34.5948)
-		(end 51.2572 34.5948)
+		(start 58.8772 34.544)
+		(end 58.8772 31.115)
 		(width 0.381)
 		(layer "F.Cu")
@@
 	)
 	(segment
-		(start 47.4472 32.6136)
-		(end 49.9364 32.6136)
+		(start 49.9872 34.5948)
+		(end 51.2572 34.5948)
 		(width 0.381)
 		(layer "F.Cu")
@@
 	)
 	(segment
-		(start 49.9364 32.6136)
-		(end 49.9364 34.5948)
+		(start 49.9872 32.4216)
+		(end 49.9872 34.5948)
 		(width 0.381)
 		(layer "F.Cu")
@@
 	)
 	(segment
-		(start 53.848 32.512)
-		(end 51.2572 32.512)
+		(start 51.2572 34.5948)
+		(end 51.2572 32.4216)
 		(width 0.381)
 		(layer "F.Cu")
@@
 	)
 	(segment
+		(start 69.2615 30.226)
+		(end 67.6402 30.226)
+		(width 0.381)
+		(layer "B.Cu")
+		(net 23)
+	)
+	(segment
 		(start 69.2844 30.2489)
-		(end 67.6402 30.2489)
+		(end 69.2615 30.226)
 		(width 0.381)
 		(layer "B.Cu")
@@
 	)
 	(segment
-		(start 67.6402 30.2489)
-		(end 67.6402 30.0739)
+		(start 69.0372 30.4961)
+		(end 69.0372 32.4216)
 		(width 0.381)
 		(layer "B.Cu")
@@
 	)
 	(segment
-		(start 69.0372 30.4961)
-		(end 69.0372 32.4216)
+		(start 70.2772 32.4216)
+		(end 70.2772 32.4358)
 		(width 0.381)
 		(layer "B.Cu")
@@
 	)
 	(segment
-		(start 70.2772 32.4216)
-		(end 70.2772 32.4358)
+		(start 67.6402 30.226)
+		(end 67.6402 30.0739)
 		(width 0.381)
 		(layer "B.Cu")
